Commit message: made it so vehicle starts at the origin and is then moved to fix issues with position of the vehicle

File: ros/src/models/gazebo/vehicle_description/urdf/body.xacro (robot description, xacro)
@@ -6,5 +6,5 @@
     <link name="base_footprint"/>
     <joint name="joint1" type="fixed" >
-      <origin xyz="${x0} ${y0} ${base_clearance}" rpy="0 0 ${psi0}" />
+      <origin xyz="0 0 ${base_clearance}" rpy="0 0 0" />
       <parent link="base_footprint" />
       <child link="${base_link}" />

File: ros/src/models/gazebo/vehicle_description/urdf/mavs.urdf.xacro (robot description, xacro)
@@ -12,8 +12,4 @@
   <xacro:property name="frameName" value="${vehicle['vehicle']['vehicle_description']['frameName']}" />
   <xacro:property name="ground_truth_topic" value="${vehicle['vehicle']['vehicle_description']['ground_truth_topic']}" />
-  <!-- initial vehicle states -->
-  <xacro:property name="x0" value="${case['case']['actual']['X0']['x']}" />
-  <xacro:property name="y0" value="${case['case']['actual']['X0']['yVal']}" />
-  <xacro:property name="psi0" value="${case['case']['actual']['X0']['psi']}" />
   <xacro:property name="scale_factor" value="${vehicle['vehicle']['vehicle_description']['scale_factor']}" />
   <xacro:property name="mesh_mode" value="${vehicle['vehicle']['vehicle_description']['mesh_mode']}"/>

Commit message: Adding changes for contact sensor

File: ros/src/models/gazebo/vehicle_description/urdf/body.xacro (robot description, xacro)
@@ -25,5 +25,5 @@
         </xacro:if>
       </visual>
-      <collision>
+      <collision name="box_collision">
         <!--selfCollide>false</selfCollide-->
         <origin xyz="0 0 ${base_height/2}" rpy="0 0 0" />

File: ros/src/models/gazebo/vehicle_description/urdf/vehicle_gazebo.urdf.xacro (robot description, xacro)
@@ -26,5 +26,13 @@
     <kp>${kp}</kp>
   </gazebo>
-  <!-- ros_control plugin -->
+  <gazebo reference="${base_link}" >
+    <sensor name="my_contact" type="contact">
+    <plugin name="contact_sensor" filename="libcontact_sensor_mavs.so">
+      <contact>
+        <collision>box_collision</collision>
+      </contact>
+   </plugin>
+ </sensor>
+</gazebo>
   <gazebo>
     <plugin name="gazebo_ros_control" filename="libgazebo_ros_control.so">

Commit message: Added contact sensor to detect collisions

File: ros/src/models/gazebo/vehicle_description/urdf/body.xacro (robot description, xacro)
@@ -25,5 +25,5 @@
         </xacro:if>
       </visual>
-      <collision name="box_collision">
+      <collision>
         <!--selfCollide>false</selfCollide-->
         <origin xyz="0 0 ${base_height/2}" rpy="0 0 0" />
@@ -41,4 +41,20 @@
       <turnGravityOff>false</turnGravityOff>
     </gazebo>
+    <gazebo reference="${base_link}" >
+      <sensor name="my_contact" type="contact">
+        <plugin name="contact_sensor" filename="libcontact_sensor_mavs.so">
+          <rosParamName>/vehicle_collided</rosParamName>
+        </plugin>
+        <contact>
+            <!-- IMPORTANT: URDF to sdf parser creates name for the collision block by itself.
+            See: http://answers.gazebosim.org/question/15095/gazebo-contact-sensor-added-to-a-robot-link-in-urdf-file-is-not-working-as-expected/
+            and: http://answers.gazebosim.org/question/12687/problems-while-parsing-gazebo-urdf-elements-with-gazebo7-and-ros-jade/
+            BE CAREFUL when renaming base_footprint link defined at top, it should be
+            updated below as well-->
+          <collision>base_footprint_fixed_joint_lump__${base_link}_collision</collision>
+        </contact>
+        <update_rate>5</update_rate>
+      </sensor>
+    </gazebo>
   </xacro:macro>
 </robot>

File: ros/src/models/gazebo/vehicle_description/urdf/vehicle_gazebo.urdf.xacro (robot description, xacro)
@@ -26,13 +26,4 @@
     <kp>${kp}</kp>
   </gazebo>
-  <gazebo reference="${base_link}" >
-    <sensor name="my_contact" type="contact">
-    <plugin name="contact_sensor" filename="libcontact_sensor_mavs.so">
-      <contact>
-        <collision>box_collision</collision>
-      </contact>
-   </plugin>
- </sensor>
-</gazebo>
   <gazebo>
     <plugin name="gazebo_ros_control" filename="libgazebo_ros_control.so">
