Commit message: created an option to use a 2D lidar

File: ros/src/models/gazebo/vehicle_description/urdf/hokuyo_laser.xacro (robot description, xacro)
@@ -1,13 +1,13 @@
 <?xml version="1.0"?>
 <robot  name="hokuyo_laser" xmlns:xacro="http://www.ros.org/wiki/xacro">
-  <xacro:macro name="hokuyo_laser" params="parent">
+  <xacro:macro name="hokuyo_laser" params="parent lidar_x lidar_z lidar_frame lidar_topic robotNamespace">
       <joint name="hokuyo_joint" type="fixed">
-        <axis xyz="0 0 ${lidar_height}" />
-        <origin xyz="0 0 ${lidar_height}" rpy="0 0 0" />
+        <axis xyz="${lidar_x} 0 ${lidar_z}" />
+        <origin xyz="${lidar_x} 0 ${lidar_z}" rpy="0 0 0" />
         <parent link="${parent}"/>
-        <child link="hokuyo_link"/>
+        <child link="${lidar_frame}"/>
      </joint>
     <!-- Hokuyo Laser -->
-    <link name="hokuyo_link">
+    <link name="${lidar_frame}">
       <collision>
         <origin xyz="0 0 0" rpy="0 0 0" />
@@ -19,5 +19,5 @@
         <origin xyz="0 0 0" rpy="0 0 0" />
         <geometry>
-          <mesh filename="package://rrbot_description/meshes/hokuyo.dae"/>
+          <mesh filename="package://velodyne_description/meshes/hokuyo.dae" />
         </geometry>
       </visual>
@@ -32,12 +32,12 @@
     <gazebo>
       <plugin name="gazebo_ros_control" filename="libgazebo_ros_control.so">
-        <robotNamespace>/bot</robotNamespace>
+        <robotNamespace>${robotNamespace}</robotNamespace>
         <robotSimType>gazebo_ros_control/DefaultRobotHWSim</robotSimType>
-        <topicName>/bot/control</topicName>
+        <topicName>/${robotNamespace}/control</topicName>
         <frameName>gazebo_control</frameName>
       </plugin>
     </gazebo>
     <!-- hokuyo -->
-    <gazebo reference="hokuyo_link">
+    <gazebo reference="${lidar_frame}">
       <sensor type="gpu_ray" name="head_hokuyo_sensor">
         <pose>0 0 0 0 0 0</pose>
@@ -47,5 +47,5 @@
           <scan>
             <horizontal>
-              <samples>720</samples>
+              <samples>1875</samples>
               <resolution>1</resolution>
               <min_angle>-1.570796</min_angle>
@@ -55,5 +55,5 @@
           <range>
             <min>0.10</min>
-            <max>30.0</max>
+            <max>100.0</max>
             <resolution>0.01</resolution>
           </range>
@@ -69,6 +69,7 @@
         </ray>
         <plugin name="gazebo_ros_head_hokuyo_controller" filename="libgazebo_ros_gpu_laser.so">
-          <topicName>/rrbot/laser/scan</topicName>
-          <frameName>hokuyo_link</frameName>
+          <!--topicName>/rrbot/laser/scan</topicName-->
+          <topicName>${lidar_topic}</topicName>
+          <frameName>${lidar_frame}</frameName>
         </plugin>
       </sensor>

File: ros/src/models/gazebo/vehicle_description/urdf/mavs.urdf.xacro (robot description, xacro)
@@ -14,4 +14,5 @@
   <xacro:property name="scale_factor" value="${vehicle['vehicle']['vehicle_description']['scale_factor']}" />
   <xacro:property name="mesh_mode" value="${vehicle['vehicle']['vehicle_description']['mesh_mode']}"/>
+  <xacro:property name="lidar_model" value="${vehicle['vehicle']['vehicle_description']['lidar_model']}"/>
   <!-- Vehicle geometry -->
   <xacro:property name="base_link" value="${vehicle['vehicle']['vehicle_description']['base_link']}" />
@@ -39,10 +40,18 @@
   <xacro:property name="lidar_z" value="${vehicle['vehicle']['vehicle_description']['lidar_z']}"/>
   <xacro:property name="lidar_x" value="${vehicle['vehicle']['vehicle_description']['lidar_x']}"/>
-  <xacro:property name="topic" value="${vehicle['vehicle']['vehicle_description']['topic']}"/>
+  <xacro:property name="lidar_frame" value="${vehicle['vehicle']['vehicle_description']['lidar_frame']}"/>
+  <xacro:property name="lidar_topic" value="${vehicle['vehicle']['vehicle_description']['lidar_topic']}"/>
+  <!--NOTE lidar_topic not currently being used -->
   <!-- Necessary includes -->
   <xacro:include filename="$(find vehicle_description)/urdf/hmmwv.xacro" />
   <xacro:include filename="$(find vehicle_description)/urdf/vehicle_gazebo.urdf.xacro" />
   <!-- Bolt-on sensors go here -->
-  <xacro:include filename="$(find vehicle_description)/urdf/velodyne_16.xacro"/>
-  <velodyne_16 parent="${base_link}" lidar_x="${lidar_x}" lidar_z="${lidar_z}"/>
+  <xacro:if value="${lidar_model == 1}">
+    <xacro:include filename="$(find vehicle_description)/urdf/velodyne_16.xacro"/>
+    <velodyne_16 parent="${base_link}" lidar_x="${lidar_x}" lidar_z="${lidar_z}" lidar_frame="${lidar_frame}" lidar_topic="${lidar_topic}" />
+  </xacro:if>
+  <xacro:if value="${lidar_model == 2}">
+    <xacro:include filename="$(find vehicle_description)/urdf/hokuyo_laser.xacro"/>
+    <hokuyo_laser parent="${base_link}" lidar_x="${lidar_x}" lidar_z="${lidar_z}" lidar_frame="${lidar_frame}" lidar_topic="${lidar_topic}" robotNamespace="robotNamespace"/>
+  </xacro:if>
 </robot>

File: ros/src/models/gazebo/vehicle_description/urdf/velodyne_16.xacro (robot description, xacro)
@@ -1,5 +1,5 @@
 <?xml version="1.0"?>
 <robot name="velodyne_16" xmlns:xacro="http://www.ros.org/wiki/xacro" >
-  <xacro:macro name="velodyne_16" params="parent lidar_x lidar_z">
+  <xacro:macro name="velodyne_16" params="parent lidar_x lidar_z lidar_frame lidar_topic">
     <joint name="velodyne_joint" type="fixed">
       <axis xyz="${lidar_x} 0 ${lidar_z}" />
@@ -34,7 +34,7 @@
       <origin xyz="0 0 0.0377" rpy="0 0 0" />
       <parent link="velodyne_base_link" />
-      <child link="velodyne_top_link"/>
+      <child link="${lidar_frame}"/>
     </joint>
-    <link name="velodyne_top_link">
+    <link name="${lidar_frame}">
       <inertial>
         <mass value="0.1"/>
@@ -50,5 +50,5 @@
     </link>
     <!-- Gazebo requires the velodyne_gazebo_plugins package -->
-    <gazebo reference="velodyne_top_link">
+    <gazebo reference="${lidar_frame}">
       <sensor type="ray" name="velodyne_16">
         <pose>0 0 0 0 0 0</pose>
@@ -82,6 +82,6 @@
         </ray>
         <plugin name="gazebo_ros_laser_controller" filename="libgazebo_ros_velodyne_laser.so">
-          <topicName>${topic}</topicName>
-          <frameName>/velodyne_top_link</frameName>
+          <topicName>${lidar_topic}</topicName>
+          <frameName>/${lidar_frame}</frameName>
           <min_range>0.9</min_range>
           <max_range>130.0</max_range>
