Commit message: fixed vehicle_description demo and removed some old yaml files

File: ros/src/models/gazebo/vehicle_description/urdf/obstacle.urdf.xacro (robot description, xacro)
@@ -12,5 +12,5 @@
     </link>
     <joint name="base_link_joint" type="fixed">
-      <origin xyz="0.0 0 0" rpy="0 0 0" />
+      <origin xyz="0 0 0" rpy="0 0 0" />
       <parent link="base_footprint"/>
       <child link="obstacle" />

Commit message: added inertia to obstacles which fixes shaking

File: ros/src/models/gazebo/vehicle_description/urdf/obstacle.urdf.xacro (robot description, xacro)
@@ -19,6 +19,6 @@
       <inertial>
         <origin xyz="${x0[idx]} ${y0[idx]} ${length[idx]/2}" rpy="0 0 0"/>
-        <mass value="100.0" />
-        <inertia  ixx="0.0" ixy="0.0"  ixz="0.0"  iyy="0.0"  iyz="0.0"  izz="0.0" />
+        <mass value="1000.0" />
+        <inertia  ixx="200.0" ixy="0.0"  ixz="0.0"  iyy="200.0"  iyz="0.0"  izz="200.0" />
       </inertial>
       <visual>

Commit message: increased the moment of inertia and mass of obstacles, there were stocastic cases when the obstacles did not follow the commands that were provided to them. These cases are fixed.

File: ros/src/models/gazebo/vehicle_description/urdf/obstacle.urdf.xacro (robot description, xacro)
@@ -19,6 +19,6 @@
       <inertial>
         <origin xyz="${x0[idx]} ${y0[idx]} ${length[idx]/2}" rpy="0 0 0"/>
-        <mass value="1000.0" />
-        <inertia  ixx="200.0" ixy="0.0"  ixz="0.0"  iyy="200.0"  iyz="0.0"  izz="200.0" />
+        <mass value="100000.0" />
+        <inertia  ixx="20000.0" ixy="0.0"  ixz="0.0"  iyy="20000.0"  iyz="0.0"  izz="20000.0" />
       </inertial>
       <visual>
